File: DRC_POWER2026.kicad_pcb (KiCad board)
At the start: 4 copper layers, 100 x 100 mm, 102 parts, among them J1 Conn_01x02, J10 VOUT, J11 P_LIGHT, J12 EMG, J2 Conn_01x02, J3 USB_C_Receptacle_USB2.0_16P, J7 VOUT, J8 P_LIGHT, K2 G5V-2, K3 G5V-2, Q1 DTC143E, SW1 RESET, U1 TLP172AM, U10 A31ASPxxVDC2D, U13 ACS772KCB-150B-PFF-T, U14 R7FA4M1AB3CFM_AA0, U15 OSL10326-L, U16 OSL10326-L, U17 OSL10326-L, U18 OSL10326-L, U19 OSL10326-L, U20 OSL10326-L, U21 OSL10326-L, U22 OSL10326-L, U23 OSL10326-L, U24 OSL10326-L, U25 OSL10326-L, U26 TM1640, U3 BP5293-50, U5 OSL10326-L, U6 A31ASPxxVDC2D, U7 TLP172AM, U8 TLP172AM, U9 ACS772KCB-150B-PFF-T

Commit message: Third commit
Other:
- board text added: "IN 12V"
- board text added: "IN 24V"
- board text added: "OUT 12V"
- board text added: "OUT 24V"
Changed lines of the file:
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@@
 		)
 	)
+	(gr_text "OUT 24V"
+		(at 55.88 -37.361866 0)
+		(layer "F.SilkS")
+		(effects
+			(font
+				(size 1.5 1.5)
+				(thickness 0.3)
+				(bold yes)
+			)
+			(justify left bottom)
+		)
+	)
+	(gr_text "IN 24V"
+		(at 69.85 -90.17 0)
+		(layer "F.SilkS")
+		(effects
+			(font
+				(size 1.5 1.5)
+				(thickness 0.3)
+				(bold yes)
+			)
+			(justify left bottom)
+		)
+	)
 	(gr_text "DRC_POWER2025 Ver.1.0\n"
 		(at 96.488 -27.9125 0)
@@
 		)
 	)
+	(gr_text "IN 12V"
+		(at 123.19 -90.17 0)
+		(layer "F.SilkS")
+		(effects
+			(font
+				(size 1.5 1.5)
+				(thickness 0.3)
+				(bold yes)
+			)
+			(justify left bottom)
+		)
+	)
+	(gr_text "OUT 12V"
+		(at 139.7 -38.1 0)
+		(layer "F.SilkS")
+		(effects
+			(font
+				(size 1.5 1.5)
+				(thickness 0.3)
+				(bold yes)
+			)
+			(justify left bottom)
+		)
+	)
 	(gr_text "V  = "
 		(at 56.6674 -8.3725 0)
@@
 	)
 	(via
-		(at 127 -91.44)
+		(at 127 -92.71)
 		(size 0.8)
 		(drill 0.4)
@@
 	)
 	(via
-		(at 132.08 -91.44)
+		(at 132.08 -90.17)
 		(size 0.8)
 		(drill 0.4)
@@
 	)
 	(via
-		(at 76.2 -91.44)
+		(at 76.2 -92.71)
 		(size 0.8)
 		(drill 0.4)
@@
 	)
 	(via
-		(at 71.12 -91.44)
+		(at 68.58 -90.17)
 		(size 0.8)
 		(drill 0.4)

Commit message: 4th commit
Parts:
- G***: moved to B.Cu
- moved G*** 34.8 mm to (92.9, -50.6), turned to 180 degrees
- moved D5 1.56 mm to (132.3, -31.5)
- moved C3 1.52 mm to (136.9, -34.1)
- moved C4 1.52 mm to (137.4, -29.0)
- moved U3 1.52 mm to (134.2, -34.1)
- moved C5 1.40 mm to (136.8, -26.7)
- turned D13 to 180 degrees
- turned D14 to 180 degrees
Connections:
- D13 pad 1: Net-(D13-K) -> GND
- D13 pad 2: GND -> Net-(D13-A)
- D14 pad 1: Net-(D14-K) -> GND
- D14 pad 2: GND -> Net-(D14-A)
- R38 pad 2: Net-(D13-K) -> Net-(D13-A)
- R40 pad 2: Net-(D14-K) -> Net-(D14-A)
Routing:
- net +12V: track 162.4 -> 164.2 mm
- net GNDPWR_12v: track 36.7 -> 38.2 mm
- net +5V: track 210.7 -> 209.2 mm
- net LED: track 55.5 -> 54.0 mm
- net Net-(D14-K): vias 1 -> 0
- net Net-(D14-A): vias 0 -> 1
- net Net-(D13-K): vias 1 -> 0
- net Net-(D13-A): vias 0 -> 1
- net GND: vias 134 -> 131
Other:
- board text added: "<<OUT 24V"
- board text added: "EMG"
- board text added: "OUT 12V>>"
- board text added: "P_LIGHT"
- board text added: "made by Yassan"
- board text removed: "OUT 12V"
- board text removed: "OUT 24V"
- board text removed: "made by Yasu"
