File: DRC_POWER2026.kicad_sch (KiCad schematic)
At the start: 35 parts, among them J1 Conn_01x02, J12 EMG, J2 Conn_01x02, J3 USB_C_Receptacle_USB2.0_16P, SW1 RESET, U14 R7FA4M1AB3CFM_AA0, U3 BP5293-50

Commit message: 4th commit
Connections:
- net GND: now also D13.1 (K), D14.1 (K); no longer D13.2 (A), D14.2 (A)
- net at R40.2: now also D14.2 (A); no longer D14.1 (K)
- net at R38.2: now also D13.2 (A); no longer D13.1 (K)
Other:
- moved on the sheet: D13, D14
Changed lines of the file:
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@@
 		(lib_name "LED_Small_3")
 		(lib_id "Device:LED_Small")
-		(at 223.52 132.08 0)
+		(at 223.52 132.08 180)
 		(unit 1)
 		(body_style 1)
@@
 		(fields_autoplaced yes)
 		(property "Reference" "D14"
-			(at 223.5835 125.73 0)
+			(at 223.4565 125.73 0)
 			(show_name no)
 			(do_not_autoplace no)
@@
 		)
 		(property "Value" "LED_Small"
-			(at 223.5835 128.27 0)
+			(at 223.4565 128.27 0)
 			(show_name no)
 			(do_not_autoplace no)
@@
 		(lib_name "LED_Small_2")
 		(lib_id "Device:LED_Small")
-		(at 223.52 123.19 0)
+		(at 223.52 123.19 180)
 		(unit 1)
 		(body_style 1)
@@
 		(fields_autoplaced yes)
 		(property "Reference" "D13"
-			(at 223.5835 116.84 0)
+			(at 223.4565 116.84 0)
 			(show_name no)
 			(do_not_autoplace no)
@@
 		)
 		(property "Value" "LED_Small"
-			(at 223.5835 119.38 0)
-			(show_name no)
-			(do_not_autoplace no)
+			(at 223.4565 119.38 0)
+			(show_name no)
+			(do_not_autoplace no)
